File: KICAD/PHORI_2_0_5.kicad_pcb (KiCad board)
At the start: 2 copper layers, 125 x 80.9 mm, 113 parts, among them J1 Conn_01x06_Female, J2 Conn_01x02, J2 Conn_01x04_Female, J4 Conn_01x01, J4 Conn_01x04_Male, J5 Rumble, J6 PinSocket_1x04_P2.00mm_Vertic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, J9 USB_B_Micro, Q1 Q_NMOS_GSD, Q2 Q_PMOS_GDS, Q3 Q_NMOS_GSD, SW1 A, SW10 Dup, SW11 Dright, SW2 B, SW4 Y, SW5 Start, SW6 L, SW7 R, SW8 Z, U1 MCP3002, U10 DRV5055Z3QDBZT, U11 DRV5055Z3QDBZT, U12 USBLC6-2P6, U13 USBLC6-2P6, U2 Stickbox_Assembly_Main, U5 Stickbox_Assembly, U6 AMS1117-3.3, U7 W25Q128JVS, U8 RP2040, Y1 Crystal_GND24

Commit message: Updated JLC files
Parts:
- moved U11 0.29 mm to (188.5, 114.9)
Changed lines of the file:
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@@
   )
   (footprint "PhobGCC_2_0_0_footprints:SOT-23" (layer "F.Cu")
-    (at 188.696875 115.095438)
+    (at 188.466397 114.924301)
     (descr "SOT, 3 Pin (https://www.jedec.org/system/files/docs/to-236h.pdf variant AB), generated with kicad-footprint-generator ipc_gullwing_generator.py")
     (tags "SOT TO_SOT_SMD")
@@
   )
   (footprint "PhobGCC_2_0_0_footprints:SOT-23" (layer "F.Cu")
-    (at 197.410875 106.204438 -90)
+    (at 197.434127 106.189462 -90)
     (descr "SOT, 3 Pin (https://www.jedec.org/system/files/docs/to-236h.pdf variant AB), generated with kicad-footprint-generator ipc_gullwing_generator.py")
     (tags "SOT TO_SOT_SMD")
@@
   (segment (start 146.206875 60.741938) (end 146.206875 58.072636) (width 0.15) (layer "F.Cu") (net 0))
   (segment (start 129.471875 66.614438) (end 127.081875 66.614438) (width 0.3) (layer "F.Cu") (net 0))
-  (segment (start 188.049375 119.413438) (end 188.049375 116.247938) (width 0.4) (layer "F.Cu") (net 0))
   (segment (start 150.731875 70.391438) (end 150.731875 70.021048) (width 0.15) (layer "F.Cu") (net 0))
   (segment (start 147.006875 60.741938) (end 147.006875 58.003583) (width 0.15) (layer "F.Cu") (net 0))
@@
   (segment (start 150.935038 61.647675) (end 151.894075 60.688638) (width 0.15) (layer "F.Cu") (net 0))
   (segment (start 152.198875 71.661438) (end 152.356559 71.503754) (width 0.15) (layer "F.Cu") (net 0))
+  (segment (start 188.049375 119.413438) (end 188.049375 116.307279) (width 0.4) (layer "F.Cu") (net 0))
   (segment (start 163.411955 59.976822) (end 163.545257 59.979438) (width 0.3) (layer "F.Cu") (net 0))
   (segment (start 157.567875 69.340438) (end 160.361875 72.134438) (width 0.15) (layer "F.Cu") (net 0))
@@
   (segment (start 151.295934 70.725221) (end 151.025296 70.995859) (width 0.15) (layer "F.Cu") (net 0))
   (segment (start 135.406875 54.417438) (end 135.434875 54.389438) (width 0.3) (layer "F.Cu") (net 0))
-  (segment (start 188.049375 116.247938) (end 187.846875 116.045438) (width 0.4) (layer "F.Cu") (net 0))
   (segment (start 99.029375 92.599438) (end 98.959375 92.529438) (width 0.25) (layer "F.Cu") (net 0))
   (segment (start 154.230875 66.835438) (end 154.230875 68.122354) (width 0.15) (layer "F.Cu") (net 0))
@@
   (segment (start 101.209375 99.366938) (end 101.216875 99.359438) (width 0.2) (layer "F.Cu") (net 0))
   (segment (start 128.706875 67.779438) (end 128.601875 67.884438) (width 0.3) (layer "F.Cu") (net 0))
+  (segment (start 188.049375 116.307279) (end 187.616397 115.874301) (width 0.4) (layer "F.Cu") (net 0))
   (segment (start 154.183435 69.327998) (end 156.684289 69.327998) (width 0.15) (layer "F.Cu") (net 0))
   (segment (start 190.806875 104.427438) (end 191.812375 104.427438) (width 0.4) (layer "F.Cu") (net 0))

Commit message: Better BOM
Parts:
- added C32: 100n, PhobGCC_2_0_0_footprints:C_0402_1005Metric, F.Cu at (141.0, 85.3)
- moved SW7 2.39 mm to (208.8, 88.6), turned to 90 degrees
- renumbered C4 to C5, R3 to R4, U11 to U10, U11 to U3, U10 to U4
Connections:
- C1 pad 1: (no net) -> +3V3
- C1 pad 2: (no net) -> GND
- C14 pad 1: (no net) -> XIN
- C14 pad 2: (no net) -> GND
- C16 pad 1: (no net) -> +5V
- C16 pad 2: (no net) -> GND
- C17 pad 1: (no net) -> +3V3
- C17 pad 2: (no net) -> GND
- C18 pad 1: (no net) -> +3V3
- C18 pad 2: (no net) -> GND
- C19 pad 1: (no net) -> +1V1
- C19 pad 2: (no net) -> GND
- C20 pad 1: (no net) -> +1V1
- C20 pad 2: (no net) -> GND
- C21 pad 1: (no net) -> +1V1
- C21 pad 2: (no net) -> GND
- C22 pad 1: (no net) -> +3V3
- C22 pad 2: (no net) -> GND
- C23 pad 1: (no net) -> +3V3
- C23 pad 2: (no net) -> GND
- C24 pad 1: (no net) -> +3V3
- C24 pad 2: (no net) -> GND
- C25 pad 1: (no net) -> +3V3
- C25 pad 2: (no net) -> GND
- C26 pad 1: (no net) -> +3V3
- C26 pad 2: (no net) -> GND
- C27 pad 1: (no net) -> +3V3
- C27 pad 2: (no net) -> GND
- C28 pad 1: (no net) -> +3V3
- C28 pad 2: (no net) -> GND
- C29 pad 1: (no net) -> +3V3
- C29 pad 2: (no net) -> GND
- C30 pad 1: (no net) -> +3V3
- C30 pad 2: (no net) -> GND
- C31 pad 1: (no net) -> +3V3
- C31 pad 2: (no net) -> GND
- C4 pad 1: (no net) -> C_Y_Filt
- C4 pad 2: (no net) -> gnd
- C5 pad 1: (no net) -> C_X_Filt
- C5 pad 2: (no net) -> gnd
- C6 pad 1: (no net) -> Stick_filt_y
- C6 pad 2: (no net) -> GND
- C7 pad 1: (no net) -> Lanalog
- C7 pad 2: (no net) -> GND
- C8 pad 1: (no net) -> Stick_filt_x
- C8 pad 2: (no net) -> GND
- D1 pad 1: (no net) -> +3V3
- D1 pad 2: (no net) -> Net-(D1-Pad2)
- D2 pad 1: (no net) -> +5V
- D2 pad 2: (no net) -> Net-(D2-Pad2)
- D5 pad 1: (no net) -> +3V3
- D5 pad 2: (no net) -> Net-(D5-Pad2)
- F1 pad 2: (no net) -> Net-(F1-Pad2)
- J1 pad 2: (no net) -> +5V
- J1 pad 3: (no net) -> GCC_DATA
- J1 pad 4: (no net) -> GND
- J1 pad 5: (no net) -> GND
- J1 pad 6: (no net) -> GND
- J2 pad 1: (no net) -> GND (x2)
- J2 pad 2: (no net) -> V
- J2 pad 4: (no net) -> +3V3
- J4 pad 1: (no net) -> gnd (x2)
- J4 pad 3: (no net) -> C_Y_Filt
- J4 pad 4: (no net) -> vcc
- J5 pad 1: (no net) -> +5V
- J5 pad 2: (no net) -> Net-(D2-Pad2)
- J6 pad 1: (no net) -> GND
- J6 pad 2: (no net) -> GPIO15
- J6 pad 3: (no net) -> GPIO14
- J6 pad 4: (no net) -> GPIO13
- J9 pad 1: (no net) -> +5V
- J9 pad 2: (no net) -> USB_D-_Raw
- J9 pad 3: (no net) -> USB_D+_Raw
- J9 pad 5: (no net) -> GND
- J9 pad 6: (no net) -> Net-(J8-Pad6)
- Q1 pad 1: (no net) -> Net-(Q1-Pad1
- Q1 pad 2: (no net) -> GND
- Q1 pad 3: (no net) -> Net-(Q1-Pad3)
- Q2 pad 1: (no net) -> Net-(Q1-Pad3)
- Q2 pad 2: (no net) -> +5V
- Q2 pad 3: (no net) -> Net-(D2-Pad2)
- Q3 pad 1: (no net) -> Net-(Q3-Pad1)
- Q3 pad 2: (no net) -> GND
- Q3 pad 3: (no net) -> Net-(F1-Pad2)
- R1 pad 1: (no net) -> Net-(R1-Pad1)
- R1 pad 2: (no net) -> GND
- R10 pad 1: (no net) -> Net-(R10-Pad1)
- R10 pad 2: (no net) -> Ladder1
- R11 pad 1: (no net) -> Rumble
- R11 pad 2: (no net) -> Net-(Q3-Pad1)
- R12 pad 1: (no net) -> Brake
- R12 pad 2: (no net) -> Net-(Q1-Pad1
- R13 pad 1: (no net) -> Net-(Q1-Pad3)
- R13 pad 2: (no net) -> +5V
- R14 pad 1: (no net) -> GND
- R14 pad 2: (no net) -> Brake
- R15 pad 1: (no net) -> GND
- R15 pad 2: (no net) -> Rumble
- R16 pad 1: (no net) -> QSPI_SS
- R16 pad 2: (no net) -> USB_BOOT
- R17 pad 1: (no net) -> Net-(J8-Pad6)
- R17 pad 2: (no net) -> GND
- R18 pad 1: (no net) -> XOUT
- R18 pad 2: (no net) -> Net-(C15-Pad1)
- R19 pad 1: (no net) -> Net-(R19-Pad1)
- R19 pad 2: (no net) -> Ladder2
- R2 pad 1: (no net) -> Net-(R10-Pad1)
- R2 pad 2: (no net) -> Net-(R1-Pad1)
- R20 pad 1: (no net) -> USB_D+
- R20 pad 2: (no net) -> Net-(R20-Pad2)
- R21 pad 1: (no net) -> USB_D-
- R21 pad 2: (no net) -> Net-(R21-pad2)
- R24 pad 1: (no net) -> Net-(R24-Pad1)
- R24 pad 2: (no net) -> Ladder3
- R25 pad 1: (no net) -> V
- R25 pad 2: (no net) -> Ladder4
- R3 pad 1: (no net) -> C_Y_Filt
- R3 pad 2: (no net) -> H2YS
- R4 pad 1: (no net) -> C_X_Filt
- R4 pad 2: (no net) -> H2XS
- R5 pad 1: (no net) -> Stick_filt_y
- R5 pad 2: (no net) -> H1YS
- R6 pad 1: (no net) -> Stick_filt_x
- R6 pad 2: (no net) -> H1XS
- R7 pad 1: (no net) -> Net-(R19-Pad1)
- R7 pad 2: (no net) -> Net-(R10-Pad1)
- R8 pad 1: (no net) -> Net-(R24-Pad1)
- R8 pad 2: (no net) -> Net-(R19-Pad1)
- R9 pad 1: (no net) -> V
- R9 pad 2: (no net) -> Net-(R24-Pad1)
- RV1 pad 1: (no net) -> +3V3
- RV1 pad 2: (no net) -> GND
- RV1 pad 3: (no net) -> Lanalog
- RV2 pad 1: (no net) -> +3V3
- RV2 pad 2: (no net) -> GND
- RV2 pad 3: (no net) -> Ranalog
- S1 pad A: (no net) -> GND
- S1 pad B: (no net) -> GND
- S1 pad C: (no net) -> USB_BOOT
- S1 pad D: (no net) -> USB_BOOT
- SW1 pad : (no net) -> GND (x2)
- SW1 pad 1: (no net) -> X
- SW1 pad 2: (no net) -> GND (x2)
- SW1 pad 1: (no net) -> A
- SW10 pad 1: (no net) -> Dup
- SW10 pad 2: (no net) -> GND (x2)
- SW10 pad 1: (no net) -> Ddown
- SW11 pad 1: (no net) -> Dleft
- SW11 pad 2: (no net) -> GND (x2)
- SW11 pad 1: (no net) -> Dright
- SW2 pad : (no net) -> GND
- SW2 pad 1: (no net) -> B
- SW2 pad 2: (no net) -> GND
- SW4 pad : (no net) -> GND
- SW4 pad 1: (no net) -> Y
- SW4 pad 2: (no net) -> GND
- SW5 pad 1: (no net) -> Start
- SW5 pad 2: (no net) -> GND
- SW5 pad 3: (no net) -> GND
- SW6 pad 1: (no net) -> L
- SW6 pad 2: (no net) -> GND
- SW7 pad 1: (no net) -> GND
- SW7 pad 2: (no net) -> R
- SW8 pad 1: (no net) -> Z
- SW8 pad 2: (no net) -> GND
- SW8 pad 1: (no net) -> GND
- SW8 pad 2: (no net) -> LeftZ
- U1 pad 1: (no net) -> CS2
- U1 pad 2: (no net) -> C_X
- U1 pad 3: (no net) -> C_Y
- U1 pad 4: (no net) -> GND
- U1 pad 5: (no net) -> Din (x2)
- U1 pad 6: (no net) -> Dout (x2)
- U1 pad 7: (no net) -> CLK (x2)
- U1 pad 8: (no net) -> VCC
- U1 pad 8: (no net) -> +3V3
- U10 pad 1: (no net) -> vcc
- U10 pad 2: (no net) -> H2XS
- U10 pad 3: (no net) -> gnd
- U11 pad 1: (no net) -> vcc
- U11 pad 2: (no net) -> H2YS
- U11 pad 3: (no net) -> gnd
- U12 pad 1: (no net) -> USB_D-_Raw
- U12 pad 2: (no net) -> GND
- U12 pad 3: (no net) -> USB_D+_Raw
- U12 pad 4: (no net) -> USB_D+
- U12 pad 5: (no net) -> +5V
- U12 pad 6: (no net) -> USB_D-
- U13 pad 1: (no net) -> unconnected
- U13 pad 2: (no net) -> GND
- U13 pad 3: (no net) -> Net-(D5-Pad2)
- U13 pad 4: (no net) -> +3V3
- U13 pad 5: (no net) -> +5V
- U13 pad 6: (no net) -> GCC_DATA
- U3 pad 1: (no net) -> +3V3
- U3 pad 2: (no net) -> H1YS
- U3 pad 3: (no net) -> GND
- U4 pad 1: (no net) -> +3V3
- U4 pad 2: (no net) -> H1XS
- U4 pad 3: (no net) -> GND
- U6 pad 1: (no net) -> GND
- U6 pad 2: (no net) -> Net-(D1-Pad2)
- U6 pad 3: (no net) -> +5V
- U7 pad 1: (no net) -> QSPI_SS
- U7 pad 2: (no net) -> QSPI_SD1
- U7 pad 3: (no net) -> QSPI_SD2
- U7 pad 4: (no net) -> GND
- U7 pad 5: (no net) -> QSPI_SD0
- U7 pad 6: (no net) -> QSPI_SCLK
- U7 pad 7: (no net) -> QSPI_SD3
- U7 pad 8: (no net) -> +3V3
- U8 pad 1: (no net) -> +3V3
- U8 pad 10: (no net) -> +3V3
- U8 pad 11: (no net) -> Dleft
- U8 pad 12: (no net) -> Dup
- U8 pad 13: (no net) -> Ddown
- U8 pad 14: (no net) -> Dright
- U8 pad 15: (no net) -> LeftZ
- U8 pad 16: (no net) -> GPIO13
- U8 pad 17: (no net) -> GPIO14
- U8 pad 18: (no net) -> GPIO15
- U8 pad 19: (no net) -> GND
- U8 pad 2: (no net) -> Ladder1
- U8 pad 20: (no net) -> XIN
- U8 pad 21: (no net) -> XOUT
- U8 pad 22: (no net) -> +3V3
- U8 pad 23: (no net) -> +1V1
- U8 pad 24: (no net) -> SWCLK
- U8 pad 25: (no net) -> SWD
- U8 pad 26: (no net) -> RUN
- U8 pad 27: (no net) -> B
- U8 pad 28: (no net) -> A
- U8 pad 29: (no net) -> X
- U8 pad 3: (no net) -> Ladder2
- U8 pad 30: (no net) -> Y
- U8 pad 31: (no net) -> Z
- U8 pad 32: (no net) -> R
- U8 pad 33: (no net) -> +3V3
- U8 pad 34: (no net) -> L
- U8 pad 35: (no net) -> CS2
- U8 pad 36: (no net) -> CS1
- U8 pad 37: (no net) -> Rumble
- U8 pad 38: (no net) -> Ranalog
- U8 pad 39: (no net) -> Lanalog
- U8 pad 4: (no net) -> Ladder3
- U8 pad 40: (no net) -> GCC_DATA
- U8 pad 41: (no net) -> Brake
- U8 pad 42: (no net) -> +3V3
- U8 pad 43: (no net) -> +3V3
- U8 pad 44: (no net) -> +3V3
- U8 pad 45: (no net) -> +1V1
- U8 pad 46: (no net) -> Net-(R21-pad2)
- U8 pad 47: (no net) -> Net-(R20-Pad2)
- U8 pad 48: (no net) -> +3V3
- U8 pad 49: (no net) -> +3V3
- U8 pad 5: (no net) -> Ladder4
- U8 pad 50: (no net) -> +1V1
- U8 pad 51: (no net) -> QSPI_SD3
- U8 pad 52: (no net) -> QSPI_SCLK
- U8 pad 53: (no net) -> QSPI_SD0
- U8 pad 54: (no net) -> QSPI_SD2
- U8 pad 55: (no net) -> QSPI_SD1
- U8 pad 56: (no net) -> QSPI_SS
- U8 pad 6: (no net) -> Dout
- U8 pad 7: (no net) -> Start
- U8 pad 8: (no net) -> CLK
- U8 pad 9: (no net) -> Din
- Y1 pad 1: (no net) -> Net-(C15-Pad1)
- Y1 pad 2: (no net) -> GND
- Y1 pad 3: (no net) -> XIN
- Y1 pad 4: (no net) -> GND
Routing:
- net (no net): track 2507.4 -> 0.00 mm, vias 126 -> 6
- net +5V: track 0.00 -> 159.0 mm, vias 0 -> 4
- net GND: track 0.00 -> 155.6 mm, vias 0 -> 45
- net CS2: track 0.00 -> 98.6 mm, vias 0 -> 4
- net LeftZ: track 0.00 -> 95.5 mm, vias 0 -> 2
- net Dout: track 0.00 -> 94.2 mm, vias 0 -> 4
- net CLK: track 0.00 -> 92.4 mm, vias 0 -> 3
- net Din: track 0.00 -> 92.2 mm, vias 0 -> 4
- net USB_D-: track 0.00 -> 87.5 mm, vias 0 -> 2
- net USB_D+: track 0.00 -> 87.3 mm, vias 0 -> 4
- net L: track 0.00 -> 85.3 mm, vias 0 -> 2
- net Net-(D2-Pad2): track 0.00 -> 82.3 mm, vias 0 -> 2
- net +3V3: track 0.00 -> 76.6 mm, vias 0 -> 10
- net Ddown: track 0.00 -> 71.6 mm, vias 0 -> 2
- net R: track 0.00 -> 70.1 mm, vias 0 -> 1
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- added copper zone on F.Cu, net +3V3
- added copper zone on B.Cu, net GND
- added copper zone on B.Cu, net gnd
- added copper zone on F.Cu, net vcc
- removed copper zone on B.Cu, net (none)
